Commit message: feat wheel macro

File: 24_02_2022/ws/src/puzzlebot_gazebo/urdf/macros.xacro (robot description, xacro)
@@ -1,25 +1,42 @@
 <?xml version="1.0"?>
 <robot xmlns:xacro="http://www.ros.org/wiki/xacro">
-<!-- note to self: modify this to add wheel as left and right with -->
-    <xacro:macro name="box_inertia" params="m x y z">
-            <inertia
-          ixx="${m/12.0 * (y*y + z*z)}" ixy="0.0" ixz="0.0"
-          iyy="${m/12.0 * (z*z + x*x)}" iyz="0.0"
-          izz="${m/12.0 * (y*y + x*x)}"/>
-        <!--  <inertia
+  <!-- note to self: modify this to add wheel as left and right with -->
+  <xacro:macro name="box_inertia" params="m x y z">
+    <inertia ixx="${m/12.0 * (y*y + z*z)}" ixy="0.0" ixz="0.0" iyy="${m/12.0 * (z*z + x*x)}" iyz="0.0" izz="${m/12.0 * (y*y + x*x)}" />
+    <!--  <inertia
           ixx="0.001" ixy="0.0" ixz="0.0"
           iyy="0.001" iyz="0.0"
           izz="0.001"/>-->
-    </xacro:macro>
-    <xacro:macro name="wheel_inertia" params="r l m">
-              <!--<inertia  ixx="${m*(3*r*r+l*l)/12}" ixy = "0" ixz = "0"
+  </xacro:macro>
+  <xacro:macro name="wheel_inertia" params="r l m">
+    <!--<inertia  ixx="${m*(3*r*r+l*l)/12}" ixy = "0" ixz = "0"
                 iyy="${m*(3*r*r+l*l)/12}" iyz = "0"
                 izz="${m*(r*r)/2}" />-->
-              <!--  <inertia  ixx="0.00001" ixy = "0" ixz = "0"
+    <!--  <inertia  ixx="0.00001" ixy = "0" ixz = "0"
                 iyy="0.00001" iyz = "0"
                 izz="0.00001" />-->
-               <inertia  ixx="${(m/12)*(3*((r*r)+((r/4)*(r/4)))+(l*l))}" ixy="0" ixz="0"
-                iyy="${(m/12)*(3*((r*r)+((r/4)*(r/4)))+(l*l))}" iyz="0"
-                izz="${(m/2)*(r*r+(r/4)*(r/4))}" />
-    </xacro:macro>
+    <inertia ixx="${(m/12)*(3*((r*r)+((r/4)*(r/4)))+(l*l))}" ixy="0" ixz="0" iyy="${(m/12)*(3*((r*r)+((r/4)*(r/4)))+(l*l))}" iyz="0" izz="${(m/2)*(r*r+(r/4)*(r/4))}" />
+  </xacro:macro>
+  <xacro:macro name="wheel" params="name reflect">
+    <link name="${name}_wheel">
+      <visual>
+        <origin xyz="0 0 0" rpy="${reflect * PI/2} 0 0" />
+        <geometry>
+          <!-- with mesh-->
+          <mesh filename="file://${mesh_wheel}" />
+        </geometry>
+      </visual>
+      <collision>
+        <origin xyz="0 0 0 " rpy="${reflect * PI/2} 0 0" />
+        <geometry>
+          <cylinder length="${wheelHeight}" radius="${wheelRadius}" />
+        </geometry>
+      </collision>
+      <inertial>
+        <mass value="${wheelMass}" />
+        <origin xyz="0 0 0" rpy="${PI/2} 0 0" />
+        <xacro:wheel_inertia r="${wheelRadius}" l="${wheelHeight}" m="${wheelMass}" />
+      </inertial>
+    </link>
+  </xacro:macro>
 </robot>

File: 24_02_2022/ws/src/puzzlebot_gazebo/urdf/puzzlebot.xacro (robot description, xacro)
@@ -57,24 +57,6 @@
 	<!-- TASK 1a - create the shape needed for the wheel specified in  -->
 	<!--RIGHT WHEEL  -->
-	<link name="right_wheel">
-		<visual>
-			<origin xyz="0 0 0" rpy="-${PI/2} 0 0" />
-			<geometry>
-				<!-- with mesh-->
-				<mesh filename="file://${mesh_wheel}" />
-			</geometry>
-		</visual>
-		<collision>
-			<origin xyz="0 0 0 " rpy="-${PI/2} 0 0" />
-			<geometry>
-				<cylinder length="${wheelHeight}" radius="${wheelRadius}" />
-			</geometry>
-		</collision>
-		<inertial>
-			<mass value="${wheelMass}" />
-			<origin xyz="0 0 0" rpy="${PI/2} 0 0" />
-			<xacro:wheel_inertia r="${wheelRadius}" l="${wheelHeight}" m="${wheelMass}" />
-		</inertial>
-	</link>
+	<xacro:wheel name="right"  reflect="-1"/>
+	<xacro:wheel name="left" reflect="1"/>
 	<!-- TASK 1b -remember using Macros-->
 	<!-- LEFT WHEEL
@@ -89,5 +71,4 @@
 		<axis xyz="0 1 0" rpy="0 0 0" />
 	</joint>
-	<!--
 	<joint name="base_to_left_w" type="continuous">
 	  <parent link="chassis" />
@@ -96,5 +77,4 @@
 	  <axis xyz="0 1 0" rpy="0 0 0" />
 	</joint>
--->
 	<!-- TRANSMISSIONS (For a more complex model and it represents actuator attributes) -->
 </robot>
