Commit message: feat right wheel

File: 24_02_2022/ws/src/puzzlebot_gazebo/urdf/puzzlebot.xacro (robot description, xacro)
@@ -1,74 +1,93 @@
-<?xml version="1.0" ?>
+<?xml version="1.0"?>
 <!-- PuzzleBot differential drive -->
 <robot name="puzzlebot" xmlns:xacro="http://www.ros.org/wiki/xacro">
-<!-- files for gazebo costumization -->
-<xacro:include filename="$(find puzzlebot_gazebo)/urdf/parameters.xacro" />
-<xacro:include filename="$(find puzzlebot_gazebo)/urdf/macros.xacro" />
-<xacro:include filename="$(find puzzlebot_gazebo)/urdf/puzzlebot.gazebo" />
-<xacro:include filename="$(find puzzlebot_gazebo)/urdf/materials.xacro" />
-<!-- Dummy link needed to load the model properly-->
-  <link name="base_link">
-    <pose>0 0 0 0 0 0</pose>
-  </link>
-  <link name="chassis">
-    <pose>0 0 0 0 0 0</pose>
-    <visual>
-      <origin xyz="0 0 0" rpy="${PI/2} 0 ${PI/2}"/>
-          <geometry>
-          	  <mesh filename="file://${mesh_chassis}"/>
-          </geometry>
-    </visual>
-    <collision name="collision_chassis">
-    	<origin rpy="0 0 0" xyz="0 0 0"/>
-          <geometry>
-            	 <box size="${chassisX} ${chassisY} ${chassisZ}"/>
-          </geometry>
-    </collision>
-    <inertial>
-      <mass value="${chassisMass}"/>
-      <xacro:box_inertia m="${chassisMass}" x="${chassisX}" y="${chassisY}" z="${chassisZ}" />
-    </inertial>
-   <!--  caster wheel attached to frame -->
-    <collision>
-	    <origin xyz="-0.095 0 -0.0425" rpy="0 0 0"/>
-		  <geometry>
-		     <sphere radius="${casterRadius}"/>
-		  </geometry>
-		   <surface>
-	      <friction>
-	         <ode>
-	          <slip1>0.0</slip1>
-	          <slip2>0.0</slip2>
-	         </ode>
-	      </friction>
-      </surface>
-	  </collision>
-	  <visual>
-      <origin xyz="-0.095 0 -0.0425" rpy="0 0 0"/>
-          <geometry>
-          	   <sphere radius="${casterRadius}"/>
-          </geometry>
-    </visual>
-  </link>
- <joint name="base_link_to_chassis" type="fixed">
-	   <parent link="base_link"/>
-	   <child link="chassis"/>
-  </joint>
-<!-- TASK 1a - create the shape needed for the wheel specified in  -->
- <!--RIGHT WHEEL
+	<!-- files for gazebo costumization -->
+	<xacro:include filename="$(find puzzlebot_gazebo)/urdf/parameters.xacro" />
+	<xacro:include filename="$(find puzzlebot_gazebo)/urdf/macros.xacro" />
+	<xacro:include filename="$(find puzzlebot_gazebo)/urdf/puzzlebot.gazebo" />
+	<xacro:include filename="$(find puzzlebot_gazebo)/urdf/materials.xacro" />
+	<!-- Dummy link needed to load the model properly-->
+	<link name="base_link">
+		<pose>0 0 0 0 0 0</pose>
+	</link>
+	<link name="chassis">
+		<pose>0 0 0 0 0 0</pose>
+		<visual>
+			<origin xyz="0 0 0" rpy="${PI/2} 0 ${PI/2}" />
+			<geometry>
+				<mesh filename="file://${mesh_chassis}" />
+			</geometry>
+		</visual>
+		<collision name="collision_chassis">
+			<origin rpy="0 0 0" xyz="0 0 0" />
+			<geometry>
+				<box size="${chassisX} ${chassisY} ${chassisZ}" />
+			</geometry>
+		</collision>
+		<inertial>
+			<mass value="${chassisMass}" />
+			<xacro:box_inertia m="${chassisMass}" x="${chassisX}" y="${chassisY}" z="${chassisZ}" />
+		</inertial>
+		<!--  caster wheel attached to frame -->
+		<collision>
+			<origin xyz="-0.095 0 -0.0425" rpy="0 0 0" />
+			<geometry>
+				<sphere radius="${casterRadius}" />
+			</geometry>
+			<surface>
+				<friction>
+					<ode>
+						<slip1>0.0</slip1>
+						<slip2>0.0</slip2>
+					</ode>
+				</friction>
+			</surface>
+		</collision>
+		<visual>
+			<origin xyz="-0.095 0 -0.0425" rpy="0 0 0" />
+			<geometry>
+				<sphere radius="${casterRadius}" />
+			</geometry>
+		</visual>
+	</link>
+	<joint name="base_link_to_chassis" type="fixed">
+		<parent link="base_link" />
+		<child link="chassis" />
+	</joint>
+	<!-- TASK 1a - create the shape needed for the wheel specified in  -->
+	<!--RIGHT WHEEL  -->
 	<link name="right_wheel">
-	</link> -->
-<!-- TASK 1b -remember using Macros-->
-<!-- LEFT WHEEL
+		<visual>
+			<origin xyz="0 0 0" rpy="-${PI/2} 0 0" />
+			<geometry>
+				<!-- with mesh-->
+				<mesh filename="file://${mesh_wheel}" />
+			</geometry>
+		</visual>
+		<collision>
+			<origin xyz="0 0 0 " rpy="-${PI/2} 0 0" />
+			<geometry>
+				<cylinder length="${wheelHeight}" radius="${wheelRadius}" />
+			</geometry>
+		</collision>
+		<inertial>
+			<mass value="${wheelMass}" />
+			<origin xyz="0 0 0" rpy="${PI/2} 0 0" />
+			<xacro:wheel_inertia r="${wheelRadius}" l="${wheelHeight}" m="${wheelMass}" />
+		</inertial>
+	</link>
+	<!-- TASK 1b -remember using Macros-->
+	<!-- LEFT WHEEL
 	<link name="left_wheel">
 	</link> -->
-<!-- Remove comment to add joint -->
-<!-- JOINTS
-  <joint name="base_to_right_w" type="continuous">
-	  <parent link="chassis" />
-	  <child link="right_wheel" />
-	  <origin xyz="0.05 -0.09 0.0" />
+	<!-- Remove comment to add joint -->
+	<!-- JOINTS  -->
+	<joint name="base_to_right_w" type="continuous">
+		<parent link="chassis" />
+		<child link="right_wheel" />
+		<origin xyz="0.05 -0.09 0.0" />
 		<axis xyz="0 1 0" rpy="0 0 0" />
 	</joint>
+	<!--
 	<joint name="base_to_left_w" type="continuous">
 	  <parent link="chassis" />
@@ -78,4 +97,4 @@
 	</joint>
 -->
-<!-- TRANSMISSIONS (For a more complex model and it represents actuator attributes) -->
+	<!-- TRANSMISSIONS (For a more complex model and it represents actuator attributes) -->
 </robot>

Commit message: feat transmissions

File: 24_02_2022/ws/src/puzzlebot_gazebo/urdf/puzzlebot.xacro (robot description, xacro)
@@ -57,6 +57,6 @@
 	<!-- TASK 1a - create the shape needed for the wheel specified in  -->
 	<!--RIGHT WHEEL  -->
-	<xacro:wheel name="right"  reflect="-1"/>
-	<xacro:wheel name="left" reflect="1"/>
+	<xacro:wheel name="right" reflect="-1" />
+	<xacro:wheel name="left" reflect="1" />
 	<!-- TASK 1b -remember using Macros-->
 	<!-- LEFT WHEEL
@@ -72,9 +72,29 @@
 	</joint>
 	<joint name="base_to_left_w" type="continuous">
-	  <parent link="chassis" />
-	  <child link="left_wheel" />
-	  <origin xyz="0.05 0.09 0" />
-	  <axis xyz="0 1 0" rpy="0 0 0" />
+		<parent link="chassis" />
+		<child link="left_wheel" />
+		<origin xyz="0.05 0.09 0" />
+		<axis xyz="0 1 0" rpy="0 0 0" />
 	</joint>
 	<!-- TRANSMISSIONS (For a more complex model and it represents actuator attributes) -->
+	<transmission name="right_wheel_trans">
+		<type>transmission_interface/SimpleTransmission</type>
+		<joint name="base_to_right_w">
+			<hardwareInterface>hardware_interface/VelocityJointInterface</hardwareInterface>
+		</joint>
+		<actuator name="right_wheel_motor">
+			<mechanicalReduction>34</mechanicalReduction>
+			<hardwareInterface>hardware_interface/VelocityJointInterface</hardwareInterface>
+		</actuator>
+	</transmission>
+	<transmission name="left_wheel_trans">
+		<type>transmission_interface/SimpleTransmission</type>
+		<joint name="base_to_left_w">
+			<hardwareInterface>hardware_interface/VelocityJointInterface</hardwareInterface>
+		</joint>
+		<actuator name="left_wheel_motor">
+			<mechanicalReduction>34</mechanicalReduction>
+			<hardwareInterface>hardware_interface/VelocityJointInterface</hardwareInterface>
+		</actuator>
+	</transmission>
 </robot>
